Commit message: fixed colors and position

File: my_rb1_description/urdf/my_rb1_robot.urdf (robot description, URDF)
Before this commit: robot RB1, 7 links, 6 joints
Links:
- added link support_chaster_wheel_back, mass 0.5; collision sphere radius=0.03; visual sphere radius=0.03
- added link support_chaster_wheel_front, mass 0.5; collision sphere radius=0.03; visual sphere radius=0.03
- link chaster_wheel_back: mass 0.5 -> None; geometry collision sphere radius=0.025; visual sphere radius=0.025
- link chaster_wheel_front: mass 0.5 -> None; geometry collision sphere radius=0.025; visual sphere radius=0.025
Joints:
- removed joint joint_base_chaster_wheel_back
- removed joint joint_base_chaster_wheel_front
- added joint joint_base_support_chaster_wheel_back: type fixed, parent base_link, child support_chaster_wheel_back, origin xyz=-0.1 0 -0.14 rpy=0 0 0, axis 0 0 0, limit effort=10000 velocity=1000
- added joint joint_base_support_chaster_wheel_front: type fixed, parent base_link, child support_chaster_wheel_front, origin xyz=0.1 0 -0.14 rpy=0 0 0, axis 0 0 0, limit effort=10000 velocity=1000
- added joint joint_chaster_wheel_front: type continuous, parent support_chaster_wheel_front, child chaster_wheel_front, origin xyz=0 0 -0.01 rpy=0 0 0, axis 0 0 1, limit effort=10000 velocity=1000
- added joint joint_support_chaster_wheel_back: type continuous, parent support_chaster_wheel_back, child chaster_wheel_back, origin xyz=0 0 -0.01 rpy=0 0 0, axis 0 0 1, limit effort=10000 velocity=1000

Commit message: final and ready for submit for second test

File: my_rb1_description/urdf/my_rb1_robot.urdf (robot description, URDF)
Before this commit: robot RB1, 9 links, 8 joints
Links:
- link link_front_laser: geometry collision cylinder length=0.020 radius=0.015; visual cylinder length=0.020 radius=0.015
Joints:
- removed joint joint_support_chaster_wheel_back
- added joint joint_chaster_wheel_back: type continuous, parent support_chaster_wheel_back, child chaster_wheel_back, origin xyz=0 0 -0.01 rpy=0 0 0, axis 0 0 1, limit effort=10000 velocity=1000

Commit message: ready for submit 3

File: my_rb1_description/urdf/my_rb1_robot.urdf (robot description, URDF)
Before this commit: robot RB1, 9 links, 8 joints
Links:
- removed link support_chaster_wheel_back
- removed link support_chaster_wheel_front
- link base_footprint: mass 25 -> 0.25
- link chaster_wheel_back: mass None -> 0.5; geometry collision sphere radius=0.025; collision sphere radius=0.03
- link chaster_wheel_front: mass None -> 0.5; geometry collision sphere radius=0.025; collision sphere radius=0.03
Joints:
- removed joint joint_base_support_chaster_wheel_back
- removed joint joint_base_support_chaster_wheel_front
- removed joint joint_chaster_wheel_back
- removed joint joint_chaster_wheel_front
- added joint joint_base_chaster_wheel_back: type fixed, parent base_link, child chaster_wheel_back, origin xyz=-0.1 0 -0.15 rpy=0 0 0, axis 0 0 0, limit effort=10000 velocity=1000
- added joint joint_base_chaster_wheel_front: type fixed, parent base_link, child chaster_wheel_front, origin xyz=0.1 0 -0.15 rpy=0 0 0, axis 0 0 0, limit effort=10000 velocity=1000

Commit message: task3 ready to submit 3

File: my_rb1_description/urdf/my_rb1_robot.urdf (robot description, URDF)
Before this commit: robot RB1, 7 links, 6 joints
Joints:
- joint joint_base_chaster_wheel_back: axis 0 0 0 -> 0 0 1
- joint joint_base_chaster_wheel_front: axis 0 0 0 -> 0 0 1
